Commit message: First pass at planning-unit test

File: trajopt_test_support/urdf/arm_around_table.urdf (robot description, URDF)
Before this commit: robot pr2, 89 links, 88 joints
Links:
- link table_link: geometry collision mesh filename=package://trajopt_test_support/meshes/table.stl; visual mesh filename=package://trajopt_test_support/meshes/table.stl

Commit message: Second pass at planning-unit test

File: trajopt_test_support/urdf/arm_around_table.urdf (robot description, URDF)
Before this commit: robot pr2, 89 links, 88 joints
Joints:
- joint table_joint: origin xyz=0.75 0 .635 rpy=0 0 0 -> xyz=1.1 0 .625 rpy=0 0 0

Commit message: MoveIt Bullet Collision Checker (Single State)

File: trajopt_test_support/urdf/arm_around_table.urdf (robot description, URDF)
Before this commit: robot pr2, 89 links, 88 joints
Links:
- link base_footprint: mass 1.0 -> None; geometry 
- link head_plate_frame: mass 0.01 -> None; geometry 
- link l_gripper_motor_accelerometer_link: mass 0.001 -> None; geometry 
- link r_gripper_motor_accelerometer_link: mass 0.001 -> None; geometry 
- link sensor_mount_link: mass 0.05 -> None; geometry 
Joints:
- joint table_joint: origin xyz=1.1 0 .625 rpy=0 0 0 -> xyz=1.11 0.0 .63 rpy=0 0 0

Commit message: Fix continuous collision checking and add original cast method

File: trajopt_test_support/urdf/arm_around_table.urdf (robot description, URDF)
Before this commit: robot pr2, 89 links, 88 joints
Joints:
- joint table_joint: origin xyz=1.11 0.0 .63 rpy=0 0 0 -> xyz=1.11 0.0 .635 rpy=0 0 0
