Commit message: Add test for objects attached to links without geometry

File: trajopt_test_support/urdf/boxbot.xacro (robot description, xacro)
@@ -10,3 +10,9 @@
     <child link="test_base_link"/>
   </joint>
+  <link name="no_geom_link"/>
+  <joint name="no_geom_joint" type="fixed">
+    <origin rpy="0 0 0" xyz="0.5 -0.5 0"/>
+    <parent link="boxbot_link"/>
+    <child link="no_geom_link"/>
+  </joint>
 </robot>
