Commit message: Rename ROSKin to ROSKinChain and add JointAccCost JointJerkCost

File: trajopt_test_support/urdf/box_1m_macro.xacro (robot description, xacro)
@@ -9,4 +9,7 @@
         <box size="1 1 1" />
       </geometry>
+      <material name="Green">
+       <color rgba="0 1.0 0.0 1.0"/>
+     </material>
     </visual>
     <collision>
