Commit message: Create custom rviz environment plugin

File: trajopt_examples/urdf/car_seat_demo_macro.xacro (robot description, xacro)
@@ -189,7 +189,7 @@
           </visual>
           <collision>
-            <origin rpy = "0 0 0" xyz="-2.900 0 0.156"/>
-            <geometry>
-              <box size="6.300 0.722 0.312"/>
+            <origin rpy = "0 0 0" xyz="-2.900 -1 0.125"/>
+            <geometry>
+              <box size="6.300 2.722 0.25"/>
             </geometry>
             <material name="yellow"/>
