Commit message: Add kdl_joint_kin to handle auxillary axes

File: trajopt_examples/urdf/grinder.xacro (robot description, xacro)
@@ -2,7 +2,7 @@
 <robot xmlns:xacro="http://wiki.ros.org/xacro">
   <xacro:macro name="grinder" params="prefix">
-    <link name="${prefix}grinder_frame">
+    <link name="${prefix}grinder_base">
       <visual>
-       <origin xyz="0 0 0" rpy="0 3.14159 0" />
+       <origin xyz="0 0 0" rpy="0 0 0" />
         <geometry>
           <mesh filename="package://trajopt_examples/meshes/puzzle_piece/grinder_visual.dae" />
@@ -10,5 +10,5 @@
       </visual>
       <collision>
-        <origin xyz="0 0 0" rpy="0 3.14159 0" />
+        <origin xyz="0 0 0" rpy="0 0 0" />
         <geometry>
           <mesh filename="package://trajopt_examples/meshes/puzzle_piece/grinder_collision.dae" />
@@ -16,4 +16,10 @@
       </collision>
     </link>
+    <link name="${prefix}grinder_frame"/>
+    <joint name="grinder_base_to_grinder_tip" type="fixed">
+      <parent link="grinder_base"/>
+      <child link="grinder_frame"/>
+      <origin xyz="0 0 0.1" rpy="0 3.14159 0"/>
+    </joint>
   </xacro:macro>
  </robot>

File: trajopt_examples/urdf/puzzle_piece_workcell.xacro (robot description, xacro)
@@ -26,8 +26,24 @@
     <origin xyz="0 0 0.5" rpy="0 0 0"/>
   </joint>
+  <link name="link_grinder"/>
   <joint name="world_to_grinder" type="fixed">
     <parent link="world"/>
-    <child link="grinder_frame"/>
-    <origin xyz="0.35 -0.35 0.7" rpy="0 3.14159 0"/>
+    <child link="link_grinder"/>
+    <origin xyz="0.35 -0.35 0.6" rpy="0 0 0"/>
+  </joint>
+  <link name="link_grinder_1"/>
+  <joint name="joint_aux1" type="revolute">
+    <parent link="link_grinder"/>
+    <child link="link_grinder_1"/>
+    <origin xyz="0 0 0" rpy="0 0 0"/>
+    <axis xyz="0 0 1" />
+    <limit lower="-3.14159" upper="3.14159" effort="0" velocity="1.0" />
+  </joint>
+  <joint name="joint_aux2" type="revolute">
+    <parent link="link_grinder_1"/>
+    <child link="grinder_base"/>
+    <origin xyz="0 0 0" rpy="0 0 0"/>
+    <axis xyz="0 1 0" />
+    <limit lower="-0.785398" upper="0.785398" effort="0" velocity="1.0" />
   </joint>
   <joint name="table_to_robot" type="fixed">
