Commit message: Move shared data to trajopt_common

File: trajopt_common/data/arm_around_table.urdf (robot description, URDF)
Before this commit: robot pr2, 88 links, 87 joints
Links:
- added link table_link; collision mesh filename=package://trajopt_common/data/meshes/Table.stl; visual mesh filename=package://trajopt_common/data/meshes/Table.stl
- link base_footprint: mass 1.0 -> None; geometry 
- link base_link: geometry collision mesh filename=package://trajopt_common/data/pr2/meshes/base_v0/base_L.stl; visual mesh filename=package://trajopt_common/data/pr2/meshes/base_v0/base.dae
- link bl_caster_l_wheel_link: geometry collision cylinder length=0.034 radius=0.074792; visual mesh filename=package://trajopt_common/data/pr2/meshes/base_v0/wheel.dae
- link bl_caster_r_wheel_link: geometry collision cylinder length=0.034 radius=0.074792; visual mesh filename=package://trajopt_common/data/pr2/meshes/base_v0/wheel.dae
- link bl_caster_rotation_link: geometry collision mesh filename=package://trajopt_common/data/pr2/meshes/base_v0/caster_L.s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; visual mesh filename=package://trajopt_common/data/pr2/meshes/base_v0/caster.stl
- link br_caster_l_wheel_link: geometry collision cylinder length=0.034 radius=0.074792; visual mesh filename=package://trajopt_common/data/pr2/meshes/base_v0/wheel.dae
- link br_caster_r_wheel_link: geometry collision cylinder length=0.034 radius=0.074792; visual mesh filename=package://trajopt_common/data/pr2/meshes/base_v0/wheel.dae
- link br_caster_rotation_link: geometry collision mesh filename=package://trajopt_common/data/pr2/meshes/base_v0/caster_L.s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; visual mesh filename=package://trajopt_common/data/pr2/meshes/base_v0/caster.stl
- link fl_caster_l_wheel_link: geometry collision cylinder length=0.034 radius=0.074792; visual mesh filename=package://trajopt_common/data/pr2/meshes/base_v0/wheel.dae
- link fl_caster_r_wheel_link: geometry collision cylinder length=0.034 radius=0.074792; visual mesh filename=package://trajopt_common/data/pr2/meshes/base_v0/wheel.dae
- link fl_caster_rotation_link: geometry collision mesh filename=package://trajopt_common/data/pr2/meshes/base_v0/caster_L.s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; visual mesh filename=package://trajopt_common/data/pr2/meshes/base_v0/caster.stl
- link fr_caster_l_wheel_link: geometry collision cylinder length=0.034 radius=0.074792; visual mesh filename=package://trajopt_common/data/pr2/meshes/base_v0/wheel.dae
- link fr_caster_r_wheel_link: geometry collision cylinder length=0.034 radius=0.074792; visual mesh filename=package://trajopt_common/data/pr2/meshes/base_v0/wheel.dae
- link fr_caster_rotation_link: geometry collision mesh filename=package://trajopt_common/data/pr2/meshes/base_v0/caster_L.s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; visual mesh filename=package://trajopt_common/data/pr2/meshes/base_v0/caster.stl
- link head_pan_link: geometry collision mesh filename=package://trajopt_common/data/pr2/meshes/head_v0/head_pan_L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; visual mesh filename=package://trajopt_common/data/pr2/meshes/head_v0/head_pan.d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
- link head_plate_frame: mass 0.01 -> None; geometry 
- link head_tilt_link: geometry collision mesh filename=package://trajopt_common/data/pr2/meshes/head_v0/head_tilt_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; visual mesh filename=package://trajopt_common/data/pr2/meshes/head_v0/head_tilt.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
- link l_elbow_flex_link: geometry collision mesh filename=package://trajopt_common/data/pr2/meshes/upper_arm_v0/elbow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; visual mesh filename=package://trajopt_common/data/pr2/meshes/upper_arm_v0/elbow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
- link l_forearm_link: geometry collision mesh filename=package://trajopt_common/data/pr2/meshes/forearm_v0/forearm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; visual mesh filename=package://trajopt_common/data/pr2/meshes/forearm_v0/forearm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
- link l_forearm_roll_link: geometry collision mesh filename=package://trajopt_common/data/pr2/meshes/upper_arm_v0/forea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; visual mesh filename=package://trajopt_common/data/pr2/meshes/upper_arm_v0/forea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
- link l_gripper_l_finger_link: geometry collision mesh filename=package://trajopt_common/data/pr2/meshes/gripper_v0/l_finge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; visual mesh filename=package://trajopt_common/data/pr2/meshes/gripper_v0/l_finge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
- link l_gripper_l_finger_tip_link: geometry collision mesh filename=package://trajopt_common/data/pr2/meshes/gripper_v0/l_finge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; visual mesh filename=package://trajopt_common/data/pr2/meshes/gripper_v0/l_finge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
- link l_gripper_motor_accelerometer_link: mass 0.001 -> None; geometry 
- link l_gripper_palm_link: geometry collision mesh filename=package://trajopt_common/data/pr2/meshes/gripper_v0/gripper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; visual mesh filename=package://trajopt_common/data/pr2/meshes/gripper_v0/gripper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
- link l_gripper_r_finger_link: geometry collision mesh filename=package://trajopt_common/data/pr2/meshes/gripper_v0/l_finge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; visual mesh filename=package://trajopt_common/data/pr2/meshes/gripper_v0/l_finge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
- link l_gripper_r_finger_tip_link: geometry collision mesh filename=package://trajopt_common/data/pr2/meshes/gripper_v0/l_finge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; visual mesh filename=package://trajopt_common/data/pr2/meshes/gripper_v0/l_finge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
- link l_shoulder_lift_link: geometry collision mesh filename=package://trajopt_common/data/pr2/meshes/shoulder_v0/should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; visual mesh filename=package://trajopt_common/data/pr2/meshes/shoulder_v0/should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
- link l_shoulder_pan_link: geometry collision mesh filename=package://trajopt_common/data/pr2/meshes/shoulder_v0/should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; visual mesh filename=package://trajopt_common/data/pr2/meshes/shoulder_v0/should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
- link l_upper_arm_link: geometry collision mesh filename=package://trajopt_common/data/pr2/meshes/upper_arm_v0/upper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; visual mesh filename=package://trajopt_common/data/pr2/meshes/upper_arm_v0/upper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
- link l_upper_arm_roll_link: geometry collision mesh filename=package://trajopt_common/data/pr2/meshes/shoulder_v0/upper_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; visual mesh filename=package://trajopt_common/data/pr2/meshes/shoulder_v0/upper_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
- link l_wrist_flex_link: geometry collision mesh filename=package://trajopt_common/data/pr2/meshes/forearm_v0/wrist_f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; visual mesh filename=package://trajopt_common/data/pr2/meshes/forearm_v0/wrist_f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
- link l_wrist_roll_link: geometry collision mesh filename=package://trajopt_common/data/pr2/meshes/forearm_v0/wrist_r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; visual mesh filename=package://trajopt_common/data/pr2/meshes/forearm_v0/wrist_r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
- link laser_tilt_mount_link: geometry collision mesh filename=package://trajopt_common/data/pr2/meshes/tilting_laser_v0/t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; visual mesh filename=package://trajopt_common/data/pr2/meshes/tilting_laser_v0/t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
- link r_elbow_flex_link: geometry collision mesh filename=package://trajopt_common/data/pr2/meshes/upper_arm_v0/elbow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; visual mesh filename=package://trajopt_common/data/pr2/meshes/upper_arm_v0/elbow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
- link r_forearm_link: geometry collision mesh filename=package://trajopt_common/data/pr2/meshes/forearm_v0/forearm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; visual mesh filename=package://trajopt_common/data/pr2/meshes/forearm_v0/forearm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
- link r_forearm_roll_link: geometry collision mesh filename=package://trajopt_common/data/pr2/meshes/upper_arm_v0/forea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; visual mesh filename=package://trajopt_common/data/pr2/meshes/upper_arm_v0/forea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
- link r_gripper_l_finger_link: geometry collision mesh filename=package://trajopt_common/data/pr2/meshes/gripper_v0/l_finge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; visual mesh filename=package://trajopt_common/data/pr2/meshes/gripper_v0/l_finge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
- link r_gripper_l_finger_tip_link: geometry collision mesh filename=package://trajopt_common/data/pr2/meshes/gripper_v0/l_finge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; visual mesh filename=package://trajopt_common/data/pr2/meshes/gripper_v0/l_finge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
- link r_gripper_motor_accelerometer_link: mass 0.001 -> None; geometry 
- link r_gripper_palm_link: geometry collision mesh filename=package://trajopt_common/data/pr2/meshes/gripper_v0/gripper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; visual mesh filename=package://trajopt_common/data/pr2/meshes/gripper_v0/gripper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
- link r_gripper_r_finger_link: geometry collision mesh filename=package://trajopt_common/data/pr2/meshes/gripper_v0/l_finge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; visual mesh filename=package://trajopt_common/data/pr2/meshes/gripper_v0/l_finge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
- link r_gripper_r_finger_tip_link: geometry collision mesh filename=package://trajopt_common/data/pr2/meshes/gripper_v0/l_finge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; visual mesh filename=package://trajopt_common/data/pr2/meshes/gripper_v0/l_finge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
- link r_shoulder_lift_link: geometry collision mesh filename=package://trajopt_common/data/pr2/meshes/shoulder_v0/should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; visual mesh filename=package://trajopt_common/data/pr2/meshes/shoulder_v0/should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
- link r_shoulder_pan_link: geometry collision mesh filename=package://trajopt_common/data/pr2/meshes/shoulder_v0/should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; visual mesh filename=package://trajopt_common/data/pr2/meshes/shoulder_v0/should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
- link r_upper_arm_link: geometry collision mesh filename=package://trajopt_common/data/pr2/meshes/upper_arm_v0/upper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; visual mesh filename=package://trajopt_common/data/pr2/meshes/upper_arm_v0/upper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
- link r_upper_arm_roll_link: geometry collision mesh filename=package://trajopt_common/data/pr2/meshes/shoulder_v0/upper_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; visual mesh filename=package://trajopt_common/data/pr2/meshes/shoulder_v0/upper_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
- link r_wrist_flex_link: geometry collision mesh filename=package://trajopt_common/data/pr2/meshes/forearm_v0/wrist_f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; visual mesh filename=package://trajopt_common/data/pr2/meshes/forearm_v0/wrist_f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
- link r_wrist_roll_link: geometry collision mesh filename=package://trajopt_common/data/pr2/meshes/forearm_v0/wrist_r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; visual mesh filename=package://trajopt_common/data/pr2/meshes/forearm_v0/wrist_r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
- link sensor_mount_link: mass 0.05 -> None; geometry 
- link torso_lift_link: geometry collision mesh filename=package://trajopt_common/data/pr2/meshes/torso_v0/torso_lif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; visual mesh filename=package://trajopt_common/data/pr2/meshes/torso_v0/torso_lif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
Joints:
- added joint table_joint: type fixed, parent base_footprint, child table_link, origin xyz=1.11 0.0 .635 rpy=0 0 0

File: trajopt_common/data/pr2.urdf (robot description, URDF)
Before this commit: robot pr2, 89 links, 88 joints
Links:
- removed link table_link
- link base_footprint: mass None -> 1.0; geometry collision box size=0.001 0.001 0.001; visual box size=0.01 0.01 0.01
- link base_link: geometry collision mesh filename=package://trajopt_common/data/pr2/meshes/base_v0/base_L.stl; visual mesh filename=package://trajopt_common/data/pr2/meshes/base_v0/base.dae
- link bl_caster_l_wheel_link: geometry collision cylinder length=0.034 radius=0.074792; visual mesh filename=package://trajopt_common/data/pr2/meshes/base_v0/wheel.dae
- link bl_caster_r_wheel_link: geometry collision cylinder length=0.034 radius=0.074792; visual mesh filename=package://trajopt_common/data/pr2/meshes/base_v0/wheel.dae
- link bl_caster_rotation_link: geometry collision mesh filename=package://trajopt_common/data/pr2/meshes/base_v0/caster_L.s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; visual mesh filename=package://trajopt_common/data/pr2/meshes/base_v0/caster.stl
- link br_caster_l_wheel_link: geometry collision cylinder length=0.034 radius=0.074792; visual mesh filename=package://trajopt_common/data/pr2/meshes/base_v0/wheel.dae
- link br_caster_r_wheel_link: geometry collision cylinder length=0.034 radius=0.074792; visual mesh filename=package://trajopt_common/data/pr2/meshes/base_v0/wheel.dae
- link br_caster_rotation_link: geometry collision mesh filename=package://trajopt_common/data/pr2/meshes/base_v0/caster_L.s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; visual mesh filename=package://trajopt_common/data/pr2/meshes/base_v0/caster.stl
- link fl_caster_l_wheel_link: geometry collision cylinder length=0.034 radius=0.074792; visual mesh filename=package://trajopt_common/data/pr2/meshes/base_v0/wheel.dae
- link fl_caster_r_wheel_link: geometry collision cylinder length=0.034 radius=0.074792; visual mesh filename=package://trajopt_common/data/pr2/meshes/base_v0/wheel.dae
- link fl_caster_rotation_link: geometry collision mesh filename=package://trajopt_common/data/pr2/meshes/base_v0/caster_L.s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; visual mesh filename=package://trajopt_common/data/pr2/meshes/base_v0/caster.stl
- link fr_caster_l_wheel_link: geometry collision cylinder length=0.034 radius=0.074792; visual mesh filename=package://trajopt_common/data/pr2/meshes/base_v0/wheel.dae
- link fr_caster_r_wheel_link: geometry collision cylinder length=0.034 radius=0.074792; visual mesh filename=package://trajopt_common/data/pr2/meshes/base_v0/wheel.dae
- link fr_caster_rotation_link: geometry collision mesh filename=package://trajopt_common/data/pr2/meshes/base_v0/caster_L.s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; visual mesh filename=package://trajopt_common/data/pr2/meshes/base_v0/caster.stl
- link head_pan_link: geometry collision mesh filename=package://trajopt_common/data/pr2/meshes/head_v0/head_pan_L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; visual mesh filename=package://trajopt_common/data/pr2/meshes/head_v0/head_pan.d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
- link head_plate_frame: mass None -> 0.01; geometry collision box size=0.01 0.01 0.01; visual box size=0.01 0.01 0.01
- link head_tilt_link: geometry collision mesh filename=package://trajopt_common/data/pr2/meshes/head_v0/head_tilt_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; visual mesh filename=package://trajopt_common/data/pr2/meshes/head_v0/head_tilt.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
- link l_elbow_flex_link: geometry collision mesh filename=package://trajopt_common/data/pr2/meshes/upper_arm_v0/elbow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; visual mesh filename=package://trajopt_common/data/pr2/meshes/upper_arm_v0/elbow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
- link l_forearm_link: geometry collision mesh filename=package://trajopt_common/data/pr2/meshes/forearm_v0/forearm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; visual mesh filename=package://trajopt_common/data/pr2/meshes/forearm_v0/forearm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
- link l_forearm_roll_link: geometry collision mesh filename=package://trajopt_common/data/pr2/meshes/upper_arm_v0/forea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; visual mesh filename=package://trajopt_common/data/pr2/meshes/upper_arm_v0/forea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
- link l_gripper_l_finger_link: geometry collision mesh filename=package://trajopt_common/data/pr2/meshes/gripper_v0/l_finge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; visual mesh filename=package://trajopt_common/data/pr2/meshes/gripper_v0/l_finge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
- link l_gripper_l_finger_tip_link: geometry collision mesh filename=package://trajopt_common/data/pr2/meshes/gripper_v0/l_finge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; visual mesh filename=package://trajopt_common/data/pr2/meshes/gripper_v0/l_finge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
- link l_gripper_motor_accelerometer_link: mass None -> 0.001; geometry collision box size=0.001 0.001 0.001; visual box size=0.001 0.001 0.001
- link l_gripper_palm_link: geometry collision mesh filename=package://trajopt_common/data/pr2/meshes/gripper_v0/gripper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; visual mesh filename=package://trajopt_common/data/pr2/meshes/gripper_v0/gripper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
- link l_gripper_r_finger_link: geometry collision mesh filename=package://trajopt_common/data/pr2/meshes/gripper_v0/l_finge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; visual mesh filename=package://trajopt_common/data/pr2/meshes/gripper_v0/l_finge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
- link l_gripper_r_finger_tip_link: geometry collision mesh filename=package://trajopt_common/data/pr2/meshes/gripper_v0/l_finge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; visual mesh filename=package://trajopt_common/data/pr2/meshes/gripper_v0/l_finge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
- link l_shoulder_lift_link: geometry collision mesh filename=package://trajopt_common/data/pr2/meshes/shoulder_v0/should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; visual mesh filename=package://trajopt_common/data/pr2/meshes/shoulder_v0/should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
- link l_shoulder_pan_link: geometry collision mesh filename=package://trajopt_common/data/pr2/meshes/shoulder_v0/should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; visual mesh filename=package://trajopt_common/data/pr2/meshes/shoulder_v0/should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
- link l_upper_arm_link: geometry collision mesh filename=package://trajopt_common/data/pr2/meshes/upper_arm_v0/upper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; visual mesh filename=package://trajopt_common/data/pr2/meshes/upper_arm_v0/upper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
- link l_upper_arm_roll_link: geometry collision mesh filename=package://trajopt_common/data/pr2/meshes/shoulder_v0/upper_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; visual mesh filename=package://trajopt_common/data/pr2/meshes/shoulder_v0/upper_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
- link l_wrist_flex_link: geometry collision mesh filename=package://trajopt_common/data/pr2/meshes/forearm_v0/wrist_f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; visual mesh filename=package://trajopt_common/data/pr2/meshes/forearm_v0/wrist_f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
- link l_wrist_roll_link: geometry collision mesh filename=package://trajopt_common/data/pr2/meshes/forearm_v0/wrist_r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; visual mesh filename=package://trajopt_common/data/pr2/meshes/forearm_v0/wrist_r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
- link laser_tilt_mount_link: geometry collision mesh filename=package://trajopt_common/data/pr2/meshes/tilting_laser_v0/t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; visual mesh filename=package://trajopt_common/data/pr2/meshes/tilting_laser_v0/t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
- link r_elbow_flex_link: geometry collision mesh filename=package://trajopt_common/data/pr2/meshes/upper_arm_v0/elbow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; visual mesh filename=package://trajopt_common/data/pr2/meshes/upper_arm_v0/elbow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
- link r_forearm_link: geometry collision mesh filename=package://trajopt_common/data/pr2/meshes/forearm_v0/forearm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; visual mesh filename=package://trajopt_common/data/pr2/meshes/forearm_v0/forearm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
- link r_forearm_roll_link: geometry collision mesh filename=package://trajopt_common/data/pr2/meshes/upper_arm_v0/forea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; visual mesh filename=package://trajopt_common/data/pr2/meshes/upper_arm_v0/forea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
- link r_gripper_l_finger_link: geometry collision mesh filename=package://trajopt_common/data/pr2/meshes/gripper_v0/l_finge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; visual mesh filename=package://trajopt_common/data/pr2/meshes/gripper_v0/l_finge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
- link r_gripper_l_finger_tip_link: geometry collision mesh filename=package://trajopt_common/data/pr2/meshes/gripper_v0/l_finge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; visual mesh filename=package://trajopt_common/data/pr2/meshes/gripper_v0/l_finge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
- link r_gripper_motor_accelerometer_link: mass None -> 0.001; geometry collision box size=0.001 0.001 0.001; visual box size=0.001 0.001 0.001
- link r_gripper_palm_link: geometry collision mesh filename=package://trajopt_common/data/pr2/meshes/gripper_v0/gripper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; visual mesh filename=package://trajopt_common/data/pr2/meshes/gripper_v0/gripper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
- link r_gripper_r_finger_link: geometry collision mesh filename=package://trajopt_common/data/pr2/meshes/gripper_v0/l_finge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; visual mesh filename=package://trajopt_common/data/pr2/meshes/gripper_v0/l_finge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
- link r_gripper_r_finger_tip_link: geometry collision mesh filename=package://trajopt_common/data/pr2/meshes/gripper_v0/l_finge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; visual mesh filename=package://trajopt_common/data/pr2/meshes/gripper_v0/l_finge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
- link r_shoulder_lift_link: geometry collision mesh filename=package://trajopt_common/data/pr2/meshes/shoulder_v0/should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; visual mesh filename=package://trajopt_common/data/pr2/meshes/shoulder_v0/should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
- link r_shoulder_pan_link: geometry collision mesh filename=package://trajopt_common/data/pr2/meshes/shoulder_v0/should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; visual mesh filename=package://trajopt_common/data/pr2/meshes/shoulder_v0/should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
- link r_upper_arm_link: geometry collision mesh filename=package://trajopt_common/data/pr2/meshes/upper_arm_v0/upper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; visual mesh filename=package://trajopt_common/data/pr2/meshes/upper_arm_v0/upper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
- link r_upper_arm_roll_link: geometry collision mesh filename=package://trajopt_common/data/pr2/meshes/shoulder_v0/upper_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; visual mesh filename=package://trajopt_common/data/pr2/meshes/shoulder_v0/upper_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
- link r_wrist_flex_link: geometry collision mesh filename=package://trajopt_common/data/pr2/meshes/forearm_v0/wrist_f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; visual mesh filename=package://trajopt_common/data/pr2/meshes/forearm_v0/wrist_f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
- link r_wrist_roll_link: geometry collision mesh filename=package://trajopt_common/data/pr2/meshes/forearm_v0/wrist_r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; visual mesh filename=package://trajopt_common/data/pr2/meshes/forearm_v0/wrist_r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
- link sensor_mount_link: mass None -> 0.05; geometry visual box size=0.01 0.01 0.01
- link torso_lift_link: geometry collision mesh filename=package://trajopt_common/data/pr2/meshes/torso_v0/torso_lif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; visual mesh filename=package://trajopt_common/data/pr2/meshes/torso_v0/torso_lif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
Joints:
- removed joint table_joint
